File: MidiKeys_Right-SCH.brd (EAGLE design)
At the start: 100 x 80 mm, 7 parts

Commit message: added all key nets
Connections:
- net N$10 renamed KEY_D3
- net N$11 renamed KEY_E3
- net N$12 renamed KEY_G3B
- net N$13 renamed KEY_A3B
- net N$14 renamed KEY_B3B
- net N$15 renamed KEY_C4
- net N$16 renamed KEY_D4
- net N$17 renamed KEY_E4
- net N$18 renamed KEY_G4B
- net N$2 renamed KEY_D2
- net N$3 renamed KEY_E2
- net N$6 renamed KEY_G2B
- net N$7 renamed KEY_A2B
- net N$8 renamed KEY_B2B
- net N$9 renamed KEY_C3
- removed net N$1: ARDUINO_DUE1.53
- new net KEY_A2: ARDUINO_DUE1.44
- new net KEY_A3: ARDUINO_DUE1.32
- new net KEY_A4: ARDUINO_DUE1.12
- new net KEY_A4B: ARDUINO_DUE1.13
- new net KEY_B2: ARDUINO_DUE1.42
- new net KEY_B3: ARDUINO_DUE1.30
- new net KEY_B4: ARDUINO_DUE1.10
- new net KEY_B4B: ARDUINO_DUE1.11
- new net KEY_C5: ARDUINO_DUE1.9
- new net KEY_D3B: ARDUINO_DUE1.40
- new net KEY_D4B: ARDUINO_DUE1.28
- new net KEY_E2B: ARDUINO_DUE1.50
- new net KEY_E3B: ARDUINO_DUE1.38
- new net KEY_E4B: ARDUINO_DUE1.26
- new net KEY_F2: ARDUINO_DUE1.48
- new net KEY_F3: ARDUINO_DUE1.36
- new net KEY_F4: ARDUINO_DUE1.24
- new net KEY_G2: ARDUINO_DUE1.46
- new net KEY_G3: ARDUINO_DUE1.34
- new net KEY_G4: ARDUINO_DUE1.22
- net KEY_C2: now also ARDUINO_DUE1.53
- net KEY_D2B: now also ARDUINO_DUE1.52
Changed lines of the file:
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@@
 <contactref element="R1" pad="1"/>
 <contactref element="U$1" pad="SW1"/>
+<contactref element="ARDUINO_DUE1" pad="53"/>
+<wire x1="-27.94" y1="-31.75" x2="55.753" y2="-141.224" width="0" layer="19" extent="1-1"/>
 <wire x1="-41.49" y1="-8.89" x2="-27.94" y2="-31.75" width="0" layer="19" extent="1-1"/>
 </signal>
@@
 <contactref element="R2" pad="1"/>
 <contactref element="U$2" pad="SW1"/>
+<contactref element="ARDUINO_DUE1" pad="52"/>
 <wire x1="-41.49" y1="-15.24" x2="-27.94" y2="-62.23" width="0" layer="19" extent="1-1"/>
+<wire x1="53.213" y1="-141.224" x2="-27.94" y2="-62.23" width="0" layer="19" extent="1-1"/>
 </signal>
 <signal name="GND">
@@
 <wire x1="-25.4" y1="-39.37" x2="-41.49" y2="-82.55" width="0" layer="19" extent="1-1"/>
 </signal>
-<signal name="N$1">
-<contactref element="ARDUINO_DUE1" pad="53"/>
-</signal>
-<signal name="N$2">
+<signal name="KEY_D2">
 <contactref element="ARDUINO_DUE1" pad="51"/>
 </signal>
-<signal name="N$3">
+<signal name="KEY_E2">
 <contactref element="ARDUINO_DUE1" pad="49"/>
 </signal>
-<signal name="N$6">
+<signal name="KEY_G3B">
+<contactref element="ARDUINO_DUE1" pad="35"/>
+</signal>
+<signal name="KEY_A3B">
+<contactref element="ARDUINO_DUE1" pad="33"/>
+</signal>
+<signal name="KEY_B3B">
+<contactref element="ARDUINO_DUE1" pad="31"/>
+</signal>
+<signal name="KEY_C4">
+<contactref element="ARDUINO_DUE1" pad="29"/>
+</signal>
+<signal name="KEY_D4">
+<contactref element="ARDUINO_DUE1" pad="27"/>
+</signal>
+<signal name="KEY_E4">
+<contactref element="ARDUINO_DUE1" pad="25"/>
+</signal>
+<signal name="KEY_G4B">
+<contactref element="ARDUINO_DUE1" pad="23"/>
+</signal>
+<signal name="KEY_G4">
+<contactref element="ARDUINO_DUE1" pad="22"/>
+</signal>
+<signal name="KEY_F4">
+<contactref element="ARDUINO_DUE1" pad="24"/>
+</signal>
+<signal name="KEY_E4B">
+<contactref element="ARDUINO_DUE1" pad="26"/>
+</signal>
+<signal name="KEY_D4B">
+<contactref element="ARDUINO_DUE1" pad="28"/>
+</signal>
+<signal name="KEY_B3">
+<contactref element="ARDUINO_DUE1" pad="30"/>
+</signal>
+<signal name="KEY_A3">
+<contactref element="ARDUINO_DUE1" pad="32"/>
+</signal>
+<signal name="KEY_G3">
+<contactref element="ARDUINO_DUE1" pad="34"/>
+</signal>
+<signal name="KEY_F3">
+<contactref element="ARDUINO_DUE1" pad="36"/>
+</signal>
+<signal name="KEY_E3B">
+<contactref element="ARDUINO_DUE1" pad="38"/>
+</signal>
+<signal name="KEY_D3B">
+<contactref element="ARDUINO_DUE1" pad="40"/>
+</signal>
+<signal name="KEY_B2">
+<contactref element="ARDUINO_DUE1" pad="42"/>
+</signal>
+<signal name="KEY_A2">
+<contactref element="ARDUINO_DUE1" pad="44"/>
+</signal>
+<signal name="KEY_G2">
+<contactref element="ARDUINO_DUE1" pad="46"/>
+</signal>
+<signal name="KEY_E2B">
+<contactref element="ARDUINO_DUE1" pad="50"/>
+</signal>
+<signal name="KEY_A4B">
+<contactref element="ARDUINO_DUE1" pad="13"/>
+</signal>
+<signal name="KEY_A4">
+<contactref element="ARDUINO_DUE1" pad="12"/>
+</signal>
+<signal name="KEY_B4B">
+<contactref element="ARDUINO_DUE1" pad="11"/>
+</signal>
+<signal name="KEY_B4">
+<contactref element="ARDUINO_DUE1" pad="10"/>
+</signal>
+<signal name="KEY_C5">
+<contactref element="ARDUINO_DUE1" pad="9"/>
+</signal>
+<signal name="KEY_F2">
+<contactref element="ARDUINO_DUE1" pad="48"/>
+</signal>
+<signal name="KEY_G2B">
 <contactref element="ARDUINO_DUE1" pad="47"/>
 </signal>
-<signal name="N$7">
+<signal name="KEY_A2B">
 <contactref element="ARDUINO_DUE1" pad="45"/>
 </signal>
-<signal name="N$8">
+<signal name="KEY_B2B">
 <contactref element="ARDUINO_DUE1" pad="43"/>
 </signal>
-<signal name="N$9">
+<signal name="KEY_C3">
 <contactref element="ARDUINO_DUE1" pad="41"/>
 </signal>
-<signal name="N$10">
+<signal name="KEY_D3">
 <contactref element="ARDUINO_DUE1" pad="39"/>
 </signal>
-<signal name="N$11">
+<signal name="KEY_E3">
 <contactref element="ARDUINO_DUE1" pad="37"/>
 </signal>
-<signal name="N$12">
-<contactref element="ARDUINO_DUE1" pad="35"/>
-</signal>
-<signal name="N$13">
-<contactref element="ARDUINO_DUE1" pad="33"/>
-</signal>
-<signal name="N$14">
-<contactref element="ARDUINO_DUE1" pad="31"/>
-</signal>
-<signal name="N$15">
-<contactref element="ARDUINO_DUE1" pad="29"/>
-</signal>
-<signal name="N$16">
-<contactref element="ARDUINO_DUE1" pad="27"/>
-</signal>
-<signal name="N$17">
-<contactref element="ARDUINO_DUE1" pad="25"/>
-</signal>
-<signal name="N$18">
-<contactref element="ARDUINO_DUE1" pad="23"/>
-</signal>
 </signals>
