File: MidiKeys_Right-SCH.brd (EAGLE design)
At the start: 140 x 60 mm, 73 parts, among them J1 3M 8550-4500

Commit message: placed solder bridges in correct places
Parts:
- moved SB4 381.9 mm to (137.0, 20.0), flipped to the bottom, turned to 90 degrees
- moved SB3 375.0 mm to (133.0, 20.0), flipped to the bottom, turned to 90 degrees
- moved SB2 368.1 mm to (129.0, 20.0), flipped to the bottom, turned to 90 degrees
- moved SA4 355.0 mm to (117.0, 20.0), flipped to the bottom, turned to 90 degrees
- moved SA3 348.1 mm to (113.0, 20.0), flipped to the bottom, turned to 90 degrees
- moved SA2 341.2 mm to (109.0, 20.0), flipped to the bottom, turned to 90 degrees
- moved SB4B 337.6 mm to (121.0, 40.0), flipped to the bottom, turned to 270 degrees
- moved SB3B 330.9 mm to (117.0, 40.0), flipped to the bottom, turned to 270 degrees
- moved SB2B 324.2 mm to (113.0, 40.0), flipped to the bottom, turned to 270 degrees
- moved SG4 317.0 mm to (97.0, 20.0), flipped to the bottom, turned to 90 degrees
- moved SA4B 310.9 mm to (101.0, 40.0), flipped to the bottom, turned to 270 degrees
- moved SG3 310.2 mm to (93.0, 20.0), flipped to the bottom, turned to 90 degrees
- moved SA3B 304.3 mm to (97.0, 40.0), flipped to the bottom, turned to 270 degrees
- moved SG2 303.4 mm to (89.0, 20.0), flipped to the bottom, turned to 90 degrees
- moved SA2B 297.6 mm to (93.0, 40.0), flipped to the bottom, turned to 270 degrees
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- renumbered A2 to A, A2B to AB, B2 to B, B2B to BB, C2 to C, D2 to D, D2B to DB, E2 to E, E2B to EB, F2 to F, G2 to G, G2B to GB

Commit message: complete layout done
Parts:
- moved R16 293.2 mm to (124.0, 4.00), flipped to the bottom
- moved R15 283.6 mm to (124.0, 16.0), flipped to the bottom
- moved R14 266.3 mm to (104.0, 4.00), flipped to the bottom
- moved R13 256.3 mm to (104.0, 16.0), flipped to the bottom
- moved R12 240.1 mm to (84.0, 4.00), flipped to the bottom
- moved R10 219.1 mm to (64.0, 4.00), flipped to the bottom
- moved R8 199.1 mm to (44.0, 4.00), flipped to the bottom
- moved R53 192.7 mm to (114.0, 56.0), flipped to the bottom
- moved R9 185.0 mm to (64.0, 16.0), flipped to the bottom
- moved R11 181.6 mm to (84.0, 16.0), flipped to the bottom
- moved R6 180.3 mm to (24.0, 4.00), flipped to the bottom
- moved R52 178.6 mm to (94.0, 44.0), flipped to the bottom
- moved R7 170.4 mm to (44.0, 16.0), flipped to the bottom
- moved R51 167.4 mm to (94.0, 56.0), flipped to the bottom
- moved R5 158.4 mm to (24.0, 16.0), flipped to the bottom
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Routing:
- net LED_SINK_TOP: track 0.00 -> 124.9 mm
- net KEY_B4: track 0.00 -> 39.8 mm
- net KEY_B3: track 0.00 -> 38.4 mm
- net KEY_B2: track 0.00 -> 36.9 mm
- net KEY_D2B: track 0.00 -> 29.8 mm
- net KEY_D3B: track 0.00 -> 28.4 mm
- net KEY_DB: track 0.00 -> 27.6 mm
- net KEY_GB: track 0.00 -> 27.6 mm
- net KEY_BB: track 0.00 -> 27.5 mm
- net KEY_A4: track 0.00 -> 27.4 mm
- net KEY_AB: track 0.00 -> 27.3 mm
- net KEY_EB: track 0.00 -> 27.3 mm
- net KEY_D4B: track 0.00 -> 26.9 mm
- net KEY_A3: track 0.00 -> 26.0 mm
- net LED_SINK_BOTTOM: track 133.0 -> 158.1 mm
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- added copper zone on layer 1, net GND
- added copper zone on layer 16, net VCC
Other:
- board text added: "KAVE"
- board text added: "KEY201"
- board text added: "MIDIKEYS"
- board text added: "v1.1"
