File: MidiKeys_Right-SCH.sch (EAGLE design)
At the start: 116 parts, among them T1 2N2222, T2 2N2222

Commit message: removed arduino shield and transistors. added 50way idc connector and solder bridges to manually connect up the correct octave. board size now 140x60. sch done. layout started
Parts:
- removed A3, A3B, A4, A4B, B3, B3B, B4, B4B, C3, C4, C5, D3, D3B, D4, D4B, E3, E3B, E4, E4B, F3, F4, G3, G3B, G4, G4B: CHERRY-MX-LED, cherrymx:CHERRY-MX-LED
- removed ARDUINO_DUE1: U1, arduino_due_shield:ARDUINO_DUE_SHIELD
- removed R17, R19, R21, R23, R25, R27, R29, R31, R33, R35, R37, R39, R41, R43, R45, R55, R57, R59, R61, R63, R65, R67, R69, R71, R73: 10k, resistor:R-EU_R0603
- removed R18, R20, R22, R24, R26, R28, R30, R32, R34, R36, R38, R40, R42, R44, R46, R56, R58, R60, R62, R64, R66, R68, R70, R72, R74: 82R, resistor:R-EU_R0603
- removed R75, R76: 1K65, resistor:R-EU_R0603
- removed T1, T2: 2N2222, adafruit:2N2222
- added J1: (no value), con-3m-skt-header:SOCKET-50V
- added SA2, SA2B, SA3, SA3B, SA4, SA4B, SB2, SB2B, SB3, SB3B, SB4, SB4B, SC2, SC3, SC4, SD2, SD2B, SD3, SD3B, SD4, SD4B, SE2, SE2B, SE3, SE3B, SE4, SE4B, SF2, SF3, SF4, SG2, SG2B, SG3, SG3B, SG4, SG4B: (no value), jumper:SJ
Connections:
- removed net KEY_C5: ARDUINO_DUE1.9, C5.SW1, R45.1
- removed net LED_CNTRL_BOTTOM: ARDUINO_DUE1.2, R76.1
- removed net LED_CNTRL_TOP: ARDUINO_DUE1.3, R75.1
- removed net N$10: D3.LED+, R20.1
- removed net N$11: E3.LED+, R22.1
- removed net N$12: F3.LED+, R24.1
- removed net N$13: G3.LED+, R26.1
- removed net N$14: A3.LED+, R28.1
- removed net N$15: B3.LED+, R30.1
- removed net N$16: C4.LED+, R32.1
- removed net N$17: D4.LED+, R34.1
- removed net N$18: E4.LED+, R36.1
- removed net N$19: F4.LED+, R38.1
- removed net N$20: G4.LED+, R40.1
- removed net N$22: B4.LED+, R44.1
- removed net N$23: C5.LED+, R46.1
- removed net N$28: D3B.LED+, R56.1
- removed net N$29: E3B.LED+, R58.1
- removed net N$30: G3B.LED+, R60.1
- removed net N$31: A3B.LED+, R62.1
- removed net N$32: B3B.LED+, R64.1
- removed net N$33: D4B.LED+, R66.1
- removed net N$34: E4B.LED+, R68.1
- removed net N$35: G4B.LED+, R70.1
- removed net N$36: A4B.LED+, R72.1
- removed net N$37: B4B.LED+, R74.1
- removed net N$65: A2B.LED-, A3B.LED-, A4B.LED-, B2B.LED-, B3B.LED-, B4B.LED-, D2B.LED-, D3B.LED-, D4B.LED-, E2B.LED-, E3B.LED-, E4B.LED-, G2B.LED-, G3B.LED-, G4B.LED-, T2.C
- removed net N$74: A2.LED-, A3.LED-, A4.LED-, B2.LED-, B3.LED-, B4.LED-, C2.LED-, C3.LED-, C4.LED-, C5.LED-, D2.LED-, D3.LED-, D4.LED-, E2.LED-, E3.LED-, E4.LED-, F2.LED-, F3.LED-, F4.LED-, G2.LED-, G3.LED-, G4.LED-, T1.C
- removed net N$75: R75.2, T2.B
- removed net N$76: R76.2, T1.B
- removed net N$9: C3.LED+, R18.1
- new net KEY_A: A2.SW1, R13.1, SA2.1, SA4.1
- new net KEY_AB: A2B.SW1, R51.1, SA2B.1, SA4B.1
- new net KEY_B: B2.SW1, R15.1, SB2.1, SB4.1
- new net KEY_BB: B2B.SW1, R53.1, SB2B.1, SB4B.1
- new net KEY_C: C2.SW1, R1.1, SC2.1, SC3.1, SC4.1
- new net KEY_D: D2.SW1, R5.1, SD2.1, SD4.1
- new net KEY_DB: D2B.SW1, R2.1, SD2B.1, SD3B.1, SD4B.1
- new net KEY_E: E2.SW1, R7.1, SE2.1, SE4.1
- new net KEY_EB: E2B.SW1, R47.1, SE2B.1, SE4B.1
- new net KEY_F: F2.SW1, R9.1, SF2.1, SF4.1
- new net KEY_G: G2.SW1, R11.1, SG2.1, SG4.1
- new net KEY_GB: G2B.SW1, R49.1, SG2B.1, SG4B.1
- new net LED_SINK_BOTTOM: A2.LED-, B2.LED-, C2.LED-, D2.LED-, E2.LED-, F2.LED-, G2.LED-, J1.30
- new net LED_SINK_TOP: A2B.LED-, B2B.LED-, D2B.LED-, E2B.LED-, G2B.LED-, J1.27
- net GND: now also J1.19, J1.21, J1.23, J1.25, J1.28; no longer A3.SW2, A3B.SW2, A4.SW2, A4B.SW2, ARDUINO_DUE1.GND, B3.SW2, B3B.SW2, B4.SW2, B4B.SW2, C3.SW2, C4.SW2, C5.SW2, D3.SW2, D3B.SW2, D4.SW2, D4B.SW2, E3.SW2, E3B.SW2, E4.SW2, E4B.SW2, F3.SW2, F4.SW2, G3.SW2, G3B.SW2, G4.SW2, G4B.SW2, T1.E, T2.E
- net KEY_A2: now also J1.12, SA2.2; no longer A2.SW1, ARDUINO_DUE1.44, R13.1
- net KEY_A2B: now also J1.11, SA2B.2; no longer A2B.SW1, ARDUINO_DUE1.45, R51.1
- net KEY_A3: now also J1.10, SA3.2; no longer A3.SW1, ARDUINO_DUE1.32, R27.1
- net KEY_A3B: now also J1.9, SA3B.2; no longer A3B.SW1, ARDUINO_DUE1.33, R61.1
- net KEY_A4: now also J1.8, SA4.2; no longer A4.SW1, ARDUINO_DUE1.12, R41.1
- net KEY_A4B: now also J1.7, SA4B.2; no longer A4B.SW1, ARDUINO_DUE1.13, R71.1
- net KEY_B2: now also J1.6, SB2.2; no longer ARDUINO_DUE1.42, B2.SW1, R15.1
- net KEY_B2B: now also J1.5, SB2B.2; no longer ARDUINO_DUE1.43, B2B.SW1, R53.1
- net KEY_B3: now also J1.4, SB3.2; no longer ARDUINO_DUE1.30, B3.SW1, R29.1
- net KEY_B3B: now also J1.3, SB3B.2; no longer ARDUINO_DUE1.31, B3B.SW1, R63.1
- net KEY_B4: now also J1.2, SB4.2; no longer ARDUINO_DUE1.10, B4.SW1, R43.1
- net KEY_B4B: now also J1.1, SB4B.2; no longer ARDUINO_DUE1.11, B4B.SW1, R73.1
- net KEY_C2: now also J1.50, SC2.2; no longer ARDUINO_DUE1.53, C2.SW1, R1.1
- net KEY_C3: now also J1.48, SC3.2; no longer ARDUINO_DUE1.41, C3.SW1, R17.1
- net KEY_C4: now also J1.46, SC4.2; no longer ARDUINO_DUE1.29, C4.SW1, R31.1
- net KEY_D2: now also J1.44, SD2.2; no longer ARDUINO_DUE1.51, D2.SW1, R5.1
- net KEY_D2B: now also J1.49, SD2B.2; no longer ARDUINO_DUE1.52, D2B.SW1, R2.1
- net KEY_D3: now also J1.42, SD3.2; no longer ARDUINO_DUE1.39, D3.SW1, R19.1
- net KEY_D3B: now also J1.47, SD3B.2; no longer ARDUINO_DUE1.40, D3B.SW1, R55.1
- net KEY_D4: now also J1.40, SD4.2; no longer ARDUINO_DUE1.27, D4.SW1, R33.1
- net KEY_D4B: now also J1.45, SD4B.2; no longer ARDUINO_DUE1.28, D4B.SW1, R65.1
- net KEY_E2: now also J1.38, SE2.2; no longer ARDUINO_DUE1.49, E2.SW1, R7.1
- net KEY_E2B: now also J1.43, SE2B.2; no longer ARDUINO_DUE1.50, E2B.SW1, R47.1
- net KEY_E3: now also J1.36, SE3.2; no longer ARDUINO_DUE1.37, E3.SW1, R21.1
- net KEY_E3B: now also J1.41, SE3B.2; no longer ARDUINO_DUE1.38, E3B.SW1, R57.1
- net KEY_E4: now also J1.34, SE4.2; no longer ARDUINO_DUE1.25, E4.SW1, R35.1
- net KEY_E4B: now also J1.39, SE4B.2; no longer ARDUINO_DUE1.26, E4B.SW1, R67.1
- net KEY_F2: now also J1.24, SF2.2; no longer ARDUINO_DUE1.48, F2.SW1, R9.1
- net KEY_F3: now also J1.22, SF3.2; no longer ARDUINO_DUE1.36, F3.SW1, R23.1
- net KEY_F4: now also J1.20, SF4.2; no longer ARDUINO_DUE1.24, F4.SW1, R37.1
- net KEY_G2: now also J1.18, SG2.2; no longer ARDUINO_DUE1.46, G2.SW1, R11.1
- net KEY_G2B: now also J1.17, SG2B.2; no longer ARDUINO_DUE1.47, G2B.SW1, R49.1
- net KEY_G3: now also J1.16, SG3.2; no longer ARDUINO_DUE1.34, G3.SW1, R25.1
- net KEY_G3B: now also J1.15, SG3B.2; no longer ARDUINO_DUE1.35, G3B.SW1, R59.1
- net KEY_G4: now also J1.14, SG4.2; no longer ARDUINO_DUE1.22, G4.SW1, R39.1
- net KEY_G4B: now also J1.13, SG4B.2; no longer ARDUINO_DUE1.23, G4B.SW1, R69.1
- net N$21: now also J1.26; no longer A4.LED+, R42.1
- net VCC: now also J1.29, J1.31, J1.32, J1.33, J1.35, J1.37; no longer ARDUINO_DUE1.3V3, R17.2, R18.2, R19.2, R20.2, R21.2, R22.2, R23.2, R24.2, R25.2, R26.2, R27.2, R28.2, R29.2, R30.2, R31.2, R32.2, R33.2, R34.2, R35.2, R36.2, R37.2, R38.2, R39.2, R40.2, R41.2, R42.2, R43.2, R44.2, R45.2, R46.2, R55.2, R56.2, R57.2, R58.2, R59.2, R60.2, R61.2, R62.2, R63.2, R64.2, R65.2, R66.2, R67.2, R68.2, R69.2, R70.2, R71.2, R72.2, R73.2, R74.2
Other:
- moved on the sheet: A2, A2B, B2, B2B, C2, D2, D2B, E2, E2B, F2, G2, G2B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

Commit message: fixed all ERC errors and started layout.
Parts:
- J1: value (none) -> 3M 8550-4500
Connections:
- removed net N$21: J1.26
- net GND: now also J1.26
- net KEY_A: now also SA3.1
- net KEY_AB: now also SA3B.1
- net KEY_B: now also SB3.1
- net KEY_BB: now also SB3B.1
- net KEY_D: now also SD3.1
- net KEY_E: now also SE3.1
- net KEY_EB: now also SE3B.1
- net KEY_F: now also SF3.1
- net KEY_G: now also SG3.1
- net KEY_GB: now also SG3B.1
